File: ST6_TA/Assemble/Assemble.kicad_sch (KiCad schematic)
At the start: 28 parts, among them SW1 SW_PUSH, SW10 SW_PUSH, SW11 SW_PUSH, SW2 SW_PUSH, SW3 SW_PUSH, SW4 SW_PUSH, SW5 SW_PUSH, SW6 SW_PUSH, SW7 SW_PUSH, SW8 SW_PUSH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

Commit message: 基盤配線前
Parts:
- added LED10, LED7, LED8, LED9: LED_SK6812MINI-E, kbd_Parts:LED_SK6812MINI-E_BL, symbol Salicylic_kbd:LED_SK6812MINI-E
- renumbered SW11 to SW10, SW7 to SW11, SW8 to SW7, SW9 to SW8, SW10 to SW9
Connections:
- net GND: now also LED10.2 (VSS), LED7.2 (VSS), LED8.2 (VSS), LED9.2 (VSS)
- net VCC: now also LED10.4 (VDD), LED7.4 (VDD), LED8.4 (VDD), LED9.4 (VDD)
- net at LED6.1 (DOUT): now also LED7.3 (DIN)
- new net: LED10.3 (DIN), LED9.1 (DOUT)
- new net: LED8.1 (DOUT), LED9.3 (DIN)
- new net: LED7.1 (DOUT), LED8.3 (DIN)
Other:
- moved on the sheet: SW11
