File: ST6_TA/Bottom/Assemble.kicad_pcb (KiCad board)
At the start: 2 copper layers, 114.3 x 88.9 mm, 5 parts

Commit message: ファイル名変更前
Parts:
- removed the Ref** at (120.7, 184.2)
Changed lines of the file:
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@@
     (pad_to_mask_clearance 0)
     (pcbplotparams
-      (layerselection 0x00010fc_ffffffff)
+      (layerselection 0x00010f0_ffffffff)
       (plot_on_all_layers_selection 0x0000000_00000000)
       (disableapertmacros false)
@@
       (usegerberattributes true)
       (usegerberadvancedattributes true)
-      (creategerberjobfile true)
+      (creategerberjobfile false)
       (dashed_line_dash_ratio 12.000000)
       (dashed_line_gap_ratio 3.000000)
@@
       (outputformat 1)
       (mirror false)
-      (drillshape 1)
+      (drillshape 0)
       (scaleselection 1)
-      (outputdirectory "")
+      (outputdirectory "../発注/Bottom/")
     )
   )
   (net 0 "")
-  (footprint "kbd_Hole:m2_Spacer_Hole_hex" (layer "F.Cu")
-    (at 120.65 184.15)
-    (descr "Mounting Hole 2.2mm, no annular, M2")
-    (tags "mounting hole 2.2mm no annular m2")
-    (attr exclude_from_pos_files exclude_from_bom)
-    (fp_text reference "Ref**" (at 0 -3.2) (layer "F.Fab")
-        (effects (font (size 1 1) (thickness 0.15)))
-    )
-    (fp_text value "Val**" (at 0 3.2) (layer "F.Fab")
-        (effects (font (size 1 1) (thickness 0.15)))
-    )
-    (fp_line (start -2.4 0) (end -1.2 2.15)
-      (stroke (width 0.1) (type solid)) (layer "Edge.Cuts"))
-    (fp_line (start -1.2 -2.15) (end -2.4 0)
-      (stroke (width 0.1) (type solid)) (layer "Edge.Cuts"))
-    (fp_line (start -1.2 2.15) (end 1.2 2.15)
-      (stroke (width 0.1) (type solid)) (layer "Edge.Cuts"))
-    (fp_line (start 1.2 -2.15) (end -1.2 -2.15)
-      (stroke (width 0.1) (type solid)) (layer "Edge.Cuts"))
-    (fp_line (start 1.2 2.15) (end 2.4 0)
-      (stroke (width 0.1) (type solid)) (layer "Edge.Cuts"))
-    (fp_line (start 2.4 0) (end 1.2 -2.15)
-      (stroke (width 0.1) (type solid)) (layer "Edge.Cuts"))
-  )
   (footprint "kbd_Hole:m2_Screw_Hole" (layer "F.Cu")
     (at 120.65 184.15)
