File: ST6_TA/Top/Assemble.kicad_pcb (KiCad board)
At the start: 2 copper layers, 114.3 x 88.9 mm, 14 parts, among them SW1 SW_PUSH, SW10 SW_PUSH, SW2 SW_PUSH, SW3 SW_PUSH, SW4 SW_PUSH, SW5 SW_PUSH, SW6 SW_PUSH, SW7 SW_PUSH, SW8 SW_PUSH, SW9 SW_PUSH

Commit message: Top,Bottom,Assenbleのネジ穴確定
Parts:
- added Ref**: Val**, kbd_Hole:m2_Spacer_Hole_hex, F.Cu at (120.7, 184.2)
