File: ST6_TA/Top/Top.kicad_pcb (KiCad board)
At the start: 2 copper layers, 114.3 x 88.9 mm, 15 parts, among them SW1 SW_PUSH, SW10 SW_PUSH, SW2 SW_PUSH, SW3 SW_PUSH, SW4 SW_PUSH, SW5 SW_PUSH, SW6 SW_PUSH, SW7 SW_PUSH, SW8 SW_PUSH, SW9 SW_PUSH

Commit message: 発注後
Parts:
- removed the Ref** at (120.7, 184.2)
Changed lines of the file:
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@@
   (net 4 "Col3")
   (net 5 "Col4")
-  (footprint "kbd_Hole:m2_Spacer_Hole_hex" (layer "F.Cu")
-    (at 120.65 184.15)
-    (descr "Mounting Hole 2.2mm, no annular, M2")
-    (tags "mounting hole 2.2mm no annular m2")
-    (attr exclude_from_pos_files exclude_from_bom)
-    (fp_text reference "Ref**" (at 0 -3.2) (layer "F.Fab")
-        (effects (font (size 1 1) (thickness 0.15)))
-    )
-    (fp_text value "Val**" (at 0 3.2) (layer "F.Fab")
-        (effects (font (size 1 1) (thickness 0.15)))
-    )
-    (fp_line (start -2.4 0) (end -1.2 2.15)
-      (stroke (width 0.1) (type solid)) (layer "Edge.Cuts"))
-    (fp_line (start -1.2 -2.15) (end -2.4 0)
-      (stroke (width 0.1) (type solid)) (layer "Edge.Cuts"))
-    (fp_line (start -1.2 2.15) (end 1.2 2.15)
-      (stroke (width 0.1) (type solid)) (layer "Edge.Cuts"))
-    (fp_line (start 1.2 -2.15) (end -1.2 -2.15)
-      (stroke (width 0.1) (type solid)) (layer "Edge.Cuts"))
-    (fp_line (start 1.2 2.15) (end 2.4 0)
-      (stroke (width 0.1) (type solid)) (layer "Edge.Cuts"))
-    (fp_line (start 2.4 0) (end 1.2 -2.15)
-      (stroke (width 0.1) (type solid)) (layer "Edge.Cuts"))
-  )
   (footprint "kbd_SW_Hole:SW_Hole_TH_1u" (layer "F.Cu")
     (at 30.95625 138.1125)

Commit message: ソケット部分を通常のものに変更
Parts:
- SW1, SW10, SW2, SW3, SW4, SW5, SW6, SW7, SW8, SW9: footprint kbd_SW_Hole:SW_Hole_TH_1u -> kbd_SW_Hole:SW_Hole_1u
- turned SW1 to 90 degrees
